File: led_controller.kicad_sch (KiCad schematic)
At the start: 29 parts, among them IC1 ESP32-C3-MINI-1-N4X, J1 Screw_Terminal_01x02, J2 Screw_Terminal_01x02, J3 Conn_01x04_Pin, J4 Screw_Terminal_01x02, J6 Conn_01x03_Pin, Q1 AO3400A, U1 LM2596S-3.3

Commit message: Add files via upload
Parts:
- added C3: 100nF, Capacitor_SMD:C_1206_3216Metric_Pad1.33x1.80mm_HandSolder, symbol Device:C
Connections:
- net EN: now also C3.1
- net GNDREF: now also C3.2
Changed lines of the file:
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@@
 	(wire
 		(pts
-			(xy 59.69 66.04) (xy 59.69 57.15)
+			(xy 59.69 68.58) (xy 59.69 57.15)
 		)
 		(stroke
@@
 		)
 	)
+	(global_label "EN"
+		(shape input)
+		(at 55.88 88.9 90)
+		(fields_autoplaced yes)
+		(effects
+			(font
+				(size 1.27 1.27)
+			)
+			(justify left)
+		)
+		(property "Intersheetrefs" "${INTERSHEET_REFS}"
+			(at 55.88 83.4353 90)
+			(effects
+				(font
+					(size 1.27 1.27)
+				)
+				(justify left)
+				(hide yes)
+			)
+		)
+	)
 	(global_label "IO7"
 		(shape input)
@@
 	(symbol
 		(lib_id "power:GNDREF")
-		(at 59.69 66.04 0)
+		(at 59.69 68.58 0)
 		(unit 1)
 		(exclude_from_sim no)
@@
 		(fields_autoplaced yes)
 		(property "Reference" "#PWR01"
-			(at 59.69 72.39 0)
+			(at 59.69 74.93 0)
 			(effects
 				(font
@@
 		)
 		(property "Value" "GNDREF"
-			(at 59.69 71.12 0)
+			(at 59.69 73.66 0)
 			(effects
 				(font
@@
 		)
 		(property "Footprint" ""
-			(at 59.69 66.04 0)
+			(at 59.69 68.58 0)
 			(effects
 				(font
@@
 		)
 		(property "Datasheet" ""
-			(at 59.69 66.04 0)
+			(at 59.69 68.58 0)
 			(effects
 				(font
@@
 		)
 		(property "Description" "Power symbol creates a global label with name \"GNDREF\" , reference supply ground"
-			(at 59.69 66.04 0)
+			(at 59.69 68.58 0)
 			(effects
 				(font
@@
 	)
 	(symbol
+		(lib_id "Device:C")
+		(at 55.88 92.71 0)
+		(unit 1)
+		(exclude_from_sim no)
+		(in_bom yes)
+		(on_board yes)
+		(dnp no)
+		(fields_autoplaced yes)
+		(property "Reference" "C3"
+			(at 59.69 91.4399 0)
+			(effects
+				(font
+					(size 1.27 1.27)
+				)
+				(justify left)
+			)
+		)
+		(property "Value" "100nF"
+			(at 59.69 93.9799 0)
+			(effects
+				(font
+					(size 1.27 1.27)
+				)
+				(justify left)
+			)
+		)
+		(property "Footprint" "Capacitor_SMD:C_1206_3216Metric_Pad1.33x1.80mm_HandSolder"
+			(at 56.8452 96.52 0)
+			(effects
+				(font
+					(size 1.27 1.27)
+				)
+				(hide yes)
+			)
+		)
+		(property "Datasheet" "~"
+			(at 55.88 92.71 0)
+			(effects
+				(font
+					(size 1.27 1.27)
+				)
+				(hide yes)
+			)
+		)
+		(property "Description" "Unpolarized capacitor"
+			(at 55.88 92.71 0)
+			(effects
+				(font
+					(size 1.27 1.27)
+				)
+				(hide yes)
+			)
+		)
+		(pin "2"
+		)
+		(pin "1"
+		)
+		(instances
+			(project "led_controller"
+				(path "/f7384fac-022b-47e0-8e4e-5c549011b8cf"
+					(reference "C3")
+					(unit 1)
+				)
+			)
+		)
+	)
+	(symbol
 		(lib_id "power:GNDREF")
 		(at 205.74 119.38 0)
@@
 					(unit 1)
 				)
+			)
+		)
+	)
+	(symbol
+		(lib_id "power:GNDREF")
+		(at 55.88 96.52 0)
+		(unit 1)
+		(exclude_from_sim no)
+		(in_bom yes)
+		(on_board yes)
+		(dnp no)
+		(fields_autoplaced yes)
+		(property "Reference" "#PWR016"
+			(at 55.88 102.87 0)
+			(effects
+				(font
+					(size 1.27 1.27)
+				)
+				(hide yes)
+			)
+		)
+		(property "Value" "GNDREF"
+			(at 55.88 101.6 0)
+			(effects
+				(font
+					(size 1.27 1.27)
+				)
+			)
+		)
+		(property "Footprint" ""
+			(at 55.88 96.52 0)
+			(effects
+				(font
+					(size 1.27 1.27)
+				)
+				(hide yes)
+			)
+		)
+		(property "Datasheet" ""
+			(at 55.88 96.52 0)
+			(effects
+				(font
+					(size 1.27 1.27)
+				)
+				(hide yes)
+			)
+		)
+		(property "Description" "Power symbol creates a global label with name \"GNDREF\" , reference supply ground"
+			(at 55.88 96.52 0)
+			(effects
+				(font
+					(size 1.27 1.27)
+				)
+				(hide yes)
+			)
+		)
+		(pin "1"
+		)
+		(instances
+			(project "led_controller"
+				(path "/f7384fac-022b-47e0-8e4e-5c549011b8cf"
+					(reference "#PWR016")
+					(unit 1)
+				)

Commit message: Add files via upload
Parts:
- Cin1, Cout2: footprint Capacitor_SMD:C_1206_3216Metric_Pad1.33x1.80mm_HandSolder -> Capacitor_SMD:CP_Elec_6.3x5.8
Changed lines of the file:
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@@
 			)
 		)
-		(property "Footprint" "Capacitor_SMD:C_1206_3216Metric_Pad1.33x1.80mm_HandSolder"
+		(property "Footprint" "Capacitor_SMD:CP_Elec_6.3x5.8"
 			(at 110.1852 64.77 0)
 			(effects
@@
 			)
 		)
-		(property "Footprint" "Capacitor_SMD:C_1206_3216Metric_Pad1.33x1.80mm_HandSolder"
+		(property "Footprint" "Capacitor_SMD:CP_Elec_6.3x5.8"
 			(at 47.9552 59.69 0)
 			(effects

Commit message: Add files via upload
Parts:
- Cin1: footprint Capacitor_SMD:CP_Elec_6.3x5.8 -> Capacitor_SMD:CP_Elec_8x10
Changed lines of the file:
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@@
 			)
 		)
-		(property "Footprint" "Capacitor_SMD:CP_Elec_6.3x5.8"
+		(property "Footprint" "Capacitor_SMD:CP_Elec_8x10"
 			(at 47.9552 59.69 0)
 			(effects

Commit message: kicad10 and modified antenna
Parts:
- C1, C3, Cin2: footprint Capacitor_SMD:C_1206_3216Metric_Pad1.33x1.80mm_HandSolder -> (none)
- R1, R2, R3, R4, R5, R6, R7: footprint Resistor_SMD:R_1206_3216Metric_Pad1.30x1.75mm_HandSolder -> (none)
